Commit message: change LiDAR pos

File: urdf/vmecanumrover.xacro (robot description, xacro)
@@ -392,10 +392,12 @@
   <!-- LiDER  -->
   <joint name="lider_joint" type="fixed">
-    <parent link="board_front_link"/>
+    <!-- <parent link="board_front_link"/> -->
+    <parent link="base_link"/>
     <child  link="lider_link"/>
   <!-- attach upper side -->
 <!--    <origin xyz="0.042 0 0.0570" rpy="0 0 0"/> -->
   <!-- attach lower side -->
-    <origin xyz="0.042 0 -0.0570" rpy="${radians(180)} 0 0"/>
+    <!-- <origin xyz="0.042 0 &#45;0.0570" rpy="${radians(180)} 0 0"/>   -->
+    <origin xyz="0.0 0 0.4" rpy="${radians(0)} 0 0"/>
   </joint>
   <link name="lider_link">

Commit message: bug fix

File: urdf/vmecanumrover.xacro (robot description, xacro)
@@ -399,5 +399,5 @@
   <!-- attach lower side -->
     <!-- <origin xyz="0.042 0 &#45;0.0570" rpy="${radians(180)} 0 0"/>   -->
-    <origin xyz="0.0 0 0.4" rpy="${radians(0)} 0 0"/>
+    <origin xyz="0.0 0 0.4" rpy="${radians(0)} ${radians(5)} 0"/>
   </joint>
   <link name="lider_link">
@@ -419,5 +419,5 @@
   <gazebo reference="lider_link">
     <material>Gazebo/Black</material>
-    <sensor type="ray" name="lrf_sensor">
+    <sensor type="gpu_ray" name="lrf_sensor">
       <pose>0 0 0 0 0 0</pose>
       <visualize>true</visualize>
@@ -443,5 +443,5 @@
         </noise>
       </ray>
-      <plugin name="gazebo_ros_lrf_controller" filename="libgazebo_ros_laser.so">
+      <plugin name="gazebo_ros_lrf_controller" filename="libgazebo_ros_gpu_laser.so">
         <topicName>/scan</topicName>
         <frameName>laser</frameName>

Commit message: fix joycon etc

File: urdf/vmecanumrover.xacro (robot description, xacro)
@@ -396,8 +396,8 @@
     <child  link="lider_link"/>
   <!-- attach upper side -->
-<!--    <origin xyz="0.042 0 0.0570" rpy="0 0 0"/> -->
+   <!-- <origin xyz="0.042 0 0.0570" rpy="0 0 0"/> -->
   <!-- attach lower side -->
-    <!-- <origin xyz="0.042 0 &#45;0.0570" rpy="${radians(180)} 0 0"/>   -->
-    <origin xyz="0.0 0 0.4" rpy="${radians(0)} ${radians(5)} 0"/>
+    <!-- <origin xyz="0.042 0 &#45;0.0570" rpy="${radians(180)} 0 0"/> -->
+    <origin xyz="0.0 0 0.3" rpy="${radians(-10)} ${radians(0)} ${radians(0)}"/>
   </joint>
   <link name="lider_link">
@@ -422,17 +422,17 @@
       <pose>0 0 0 0 0 0</pose>
       <visualize>true</visualize>
-      <update_rate>40</update_rate>
+      <update_rate>100</update_rate>
       <ray>
         <scan>
           <horizontal>
-            <samples>1000</samples>
-            <resolution>1</resolution>
-            <min_angle>-1.57</min_angle>
-            <max_angle>1.57</max_angle>
+            <samples>1080</samples>
+            <resolution>1.5</resolution>
+            <min_angle>${radians(-135)}</min_angle>
+            <max_angle>${radians(135)}</max_angle>
           </horizontal>
         </scan>
         <range>
           <min>0.06</min>
-          <max>4.0</max>
+          <max>5.2</max>
         <resolution>0.001</resolution>
         </range>
